File: PAMI_V01.kicad_pcb (KiCad board)
At the start: 2 copper layers, 70 x 60 mm, 49 parts, among them J1 Conn_01x04, J10 Conn_01x07, J2 Conn_01x04, J20 Conn_01x03, J21 Conn_01x03, J22 Conn_01x02, J3 Conn_OLED_Screen, J4 USB_B, J5 Conn_02x02_Odd_Even, J6 Conn_02x02_Odd_Even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

Commit message: updating kicad files
Parts:
- moved J20 1.91 mm to (155.3, 120.5)
- moved J21 1.81 mm to (157.5, 113.5)
- moved D4 1.12 mm to (125.3, 111.4)
- moved J8 0.83 mm to (172.3, 93.9)
- moved U1 0.57 mm to (174.2, 123.3)
- moved J1 0.55 mm to (185.6, 127.2)
- moved C6 0.52 mm to (185.8, 134.5)
- moved R7 0.38 mm to (174.9, 99.4)
- moved H1 0.08 mm to (127.0, 93.0)
- moved R4 0.08 mm to (125.1, 103.6)
Routing:
- net GPIO1: track 39.8 -> 46.1 mm
- net GPIO9: track 10.8 -> 13.2 mm
- net GPIO10: track 11.9 -> 14.1 mm
- net GPIO11: track 13.0 -> 15.1 mm
- net GPIO47: track 3.76 -> 5.63 mm
- net GPIO14: track 3.76 -> 5.63 mm
- net GPIO12: track 3.76 -> 5.63 mm
- net GPIO35: track 32.3 -> 34.0 mm
- net GPIO7: track 19.6 -> 21.3 mm, vias 0 -> 1
- net GPIO36: track 31.5 -> 32.6 mm
- net +5V: track 150.3 -> 149.2 mm
- net Net-(U3-MTDO/GPIO40/CLK_OUT2): track 5.50 -> 6.28 mm
- net GPIO15: track 10.1 -> 9.35 mm
- net Net-(BZ1-+): track 35.6 -> 35.0 mm
- net Net-(D4-A): track 6.45 -> 7.10 mm
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Other:
- outline, holes or cut-outs redrawn

Commit message: Unishape PAMI board V2
Parts:
- added J11: Conn_HC_SR04, Connector_PinHeader_2.54mm:PinHeader_1x04_P2.54mm_Vertical, F.Cu at (157.6, 117.6)
- moved J20 36.4 mm to (190.1, 110.0), turned to 0 degrees
- moved J9 0.86 mm to (178.8, 108.7)
- moved J10 0.84 mm to (182.5, 108.7)
Connections:
- J20 pad 1: GPIO9 -> unconnected-(J20-Pin_1-Pad1)
- J20 pad 2: GPIO10 -> unconnected-(J20-Pin_2-Pad2)
- J20 pad 3: GPIO11 -> unconnected-(J20-Pin_3-Pad3)
- J21 pad 2: GPIO14 -> GPIO13
- J21 pad 3: GPIO47 -> GPIO14
- U3 pad 21: unconnected-(U3-GPIO13/TOUCH13/ADC2_CH2/FSPIQ/FSPIIO7/SUBSPIQ-Pad21) -> GPIO13
- U3 pad 24: GPIO47 -> unconnected-(U3-GPIO47/SPICLK_P/SUBSPICLK_P_DIFF-Pad24)
Routing:
- net GPIO11: track 15.1 -> 0.00 mm
- net +5V: track 149.2 -> 160.3 mm
- net GPIO47: track 5.63 -> 0.00 mm
- net GPIO13: track 0.00 -> 5.21 mm
- net GPIO9: track 13.2 -> 17.3 mm
- net GPIO1: track 46.1 -> 48.0 mm
- net +3.3V: track 140.9 -> 139.4 mm
- net SCL: track 16.7 -> 18.0 mm
- net SDA: track 17.9 -> 19.2 mm
